Commit message: update for two sonar

File: urdf/turtlebot3_burger_sonar.gazebo.xacro (robot description, xacro)
@@ -125,6 +125,6 @@
   </gazebo>
  <!-- Added for SR04 by OJ, SDF-Code in <gazebo>-Tag -->
-<gazebo reference="base_sonar_front"> <!-- same as link-->
- <sensor type="ray" name="sonar">
+<gazebo reference="base_sonar_front_left"> <!-- same as link-->
+ <sensor type="ray" name="sonar_left">
           <pose>0.25 0 0 0 0 0</pose>
           <update_rate>5</update_rate>
@@ -154,6 +154,42 @@
             <alwaysOn>true</alwaysOn>
             <updateRate>5</updateRate>
-            <topicName>sonar</topicName>
-            <frameName>base_sonar_front</frameName>  <!-- old sonar_link -->-->
+            <topicName>sonar_left</topicName>
+            <frameName>base_sonar_front_left</frameName>  <!-- old sonar_link -->-->
+            <fov>0.5</fov>
+            <radiation>ultrasound</radiation>
+          </plugin>
+        </sensor>
+  </gazebo>
+<gazebo reference="base_sonar_front_right"> <!-- same as link-->
+ <sensor type="ray" name="sonar_right">
+          <pose>0.25 0 0 0 0 0</pose>
+          <update_rate>5</update_rate>
+          <ray>
+            <scan>
+              <horizontal>
+                <samples>5</samples>
+                <resolution>1.0</resolution>
+                <min_angle>-0.25</min_angle>
+                <max_angle>0.25</max_angle>
+              </horizontal>
+              <vertical>
+                <samples>5</samples>
+                <resolution>1</resolution>
+                <min_angle>-0.25</min_angle>
+                <max_angle>0.25</max_angle>
+              </vertical>
+            </scan>
+            <range>
+              <min>0.01</min>
+              <max>0.75</max>
+              <resolution>0.01</resolution>
+            </range>
+          </ray>
+          <plugin filename="libgazebo_ros_range.so" name="gazebo_ros_range">
+            <gaussianNoise>0.005</gaussianNoise>
+            <alwaysOn>true</alwaysOn>
+            <updateRate>5</updateRate>
+            <topicName>sonar_right</topicName>
+            <frameName>base_sonar_front_right</frameName>  <!-- old sonar_link -->-->
             <fov>0.5</fov>
             <radiation>ultrasound</radiation>

File: urdf/turtlebot3_burger_sonar.urdf.xacro (robot description, xacro)
@@ -144,11 +144,34 @@
  https://github.com/ros-simulation/gazebo_ros_pkgs/blob/kinetic-devel/gazebo_plugins/test/test_worlds/gazebo_ros_range.world#L82
  -->
-    <joint name="sonar_front_joint" type="fixed">
+    <joint name="sonar_front_joint_left" type="fixed">
         <axis xyz="0 1 0" />
-        <origin rpy="0 -0.12 0" xyz="0.04 0 0.10" />
+        <origin rpy="0 -0.12 0.2" xyz="0.04 0.06 0.10" />
         <parent link="base_link"/>
-        <child link="base_sonar_front"/>
+        <child link="base_sonar_front_left"/>
     </joint>
-    <link name="base_sonar_front">
+    <link name="base_sonar_front_left">
+        <collision>
+        <origin xyz="0 0 0" rpy="0 0 0"/>
+        <geometry>
+            <box size="0.01 0.01 0.01"/>
+        </geometry>
+        </collision>    <visual>
+        <origin xyz="0 0 0" rpy="0 0 0"/>
+        <geometry>
+            <box size="0.01 0.01 0.01"/>
+        </geometry>
+        </visual>    <inertial>
+        <mass value="1e-5" />
+        <origin xyz="0 0 0" rpy="0 0 0"/>
+        <inertia ixx="1e-6" ixy="0" ixz="0" iyy="1e-6" iyz="0" izz="1e-6" />
+        </inertial>
+    </link>
+ <joint name="sonar_front_joint_right" type="fixed">
+        <axis xyz="0 1 0" />
+        <origin rpy="0 -0.12 -0.2" xyz="0.04 -0.06 0.10" />
+        <parent link="base_link"/>
+        <child link="base_sonar_front_right"/>
+    </joint>
+    <link name="base_sonar_front_right">
         <collision>
         <origin xyz="0 0 0" rpy="0 0 0"/>
