Commit message: rearrange sensors in urdf

File: urdf/turtlebot3_burger_sonar.urdf.xacro (robot description, xacro)
@@ -146,5 +146,5 @@
     <joint name="sonar_front_joint_left" type="fixed">
         <axis xyz="0 1 0" />
-        <origin rpy="0 -0.12 0.2" xyz="0.04 0.06 0.10" />
+        <origin rpy="0 0 0" xyz="0.04 0.06 0.06" />
         <parent link="base_link"/>
         <child link="base_sonar_front_left"/>
@@ -169,5 +169,5 @@
  <joint name="sonar_front_joint_right" type="fixed">
         <axis xyz="0 1 0" />
-        <origin rpy="0 -0.12 -0.2" xyz="0.04 -0.06 0.10" />
+        <origin rpy="0 0 0" xyz="0.04 -0.06 0.06" />
         <parent link="base_link"/>
         <child link="base_sonar_front_right"/>

Commit message: changes in URDF

File: urdf/turtlebot3_burger_sonar.urdf.xacro (robot description, xacro)
@@ -146,5 +146,5 @@
     <joint name="sonar_front_joint_left" type="fixed">
         <axis xyz="0 1 0" />
-        <origin rpy="0 0 0" xyz="0.04 0.06 0.06" />
+        <origin rpy="0 0 0.2" xyz="0.065 0.044 0.078" />
         <parent link="base_link"/>
         <child link="base_sonar_front_left"/>
@@ -154,10 +154,10 @@
         <origin xyz="0 0 0" rpy="0 0 0"/>
         <geometry>
-            <box size="0.01 0.01 0.01"/>
+            <box size="0.04 0.01 0.01"/>
         </geometry>
         </collision>    <visual>
         <origin xyz="0 0 0" rpy="0 0 0"/>
         <geometry>
-            <box size="0.01 0.01 0.01"/>
+            <box size="0.04 0.01 0.01"/>
         </geometry>
         </visual>    <inertial>
@@ -169,5 +169,5 @@
  <joint name="sonar_front_joint_right" type="fixed">
         <axis xyz="0 1 0" />
-        <origin rpy="0 0 0" xyz="0.04 -0.06 0.06" />
+        <origin rpy="0 0 -0.2" xyz="0.065 -0.044 0.078" />
         <parent link="base_link"/>
         <child link="base_sonar_front_right"/>
@@ -177,10 +177,10 @@
         <origin xyz="0 0 0" rpy="0 0 0"/>
         <geometry>
-            <box size="0.01 0.01 0.01"/>
+            <box size="0.04 0.01 0.01"/>
         </geometry>
         </collision>    <visual>
         <origin xyz="0 0 0" rpy="0 0 0"/>
         <geometry>
-            <box size="0.01 0.01 0.01"/>
+            <box size="0.04 0.01 0.01"/>
         </geometry>
         </visual>    <inertial>

Commit message: changed sonar position

File: urdf/turtlebot3_burger_sonar.urdf.xacro (robot description, xacro)
@@ -144,49 +144,53 @@
  https://github.com/ros-simulation/gazebo_ros_pkgs/blob/kinetic-devel/gazebo_plugins/test/test_worlds/gazebo_ros_range.world#L82
  -->
-    <joint name="sonar_front_joint_left" type="fixed">
-        <axis xyz="0 1 0" />
-        <origin rpy="0 0 0.2" xyz="0.065 0.044 0.078" />
-        <parent link="base_link"/>
-        <child link="base_sonar_front_left"/>
-    </joint>
-    <link name="base_sonar_front_left">
-        <collision>
-        <origin xyz="0 0 0" rpy="0 0 0"/>
-        <geometry>
-            <box size="0.04 0.01 0.01"/>
-        </geometry>
-        </collision>    <visual>
-        <origin xyz="0 0 0" rpy="0 0 0"/>
-        <geometry>
-            <box size="0.04 0.01 0.01"/>
-        </geometry>
-        </visual>    <inertial>
-        <mass value="1e-5" />
-        <origin xyz="0 0 0" rpy="0 0 0"/>
-        <inertia ixx="1e-6" ixy="0" ixz="0" iyy="1e-6" iyz="0" izz="1e-6" />
-        </inertial>
-    </link>
- <joint name="sonar_front_joint_right" type="fixed">
-        <axis xyz="0 1 0" />
-        <origin rpy="0 0 -0.2" xyz="0.065 -0.044 0.078" />
-        <parent link="base_link"/>
-        <child link="base_sonar_front_right"/>
-    </joint>
-    <link name="base_sonar_front_right">
-        <collision>
-        <origin xyz="0 0 0" rpy="0 0 0"/>
-        <geometry>
-            <box size="0.04 0.01 0.01"/>
-        </geometry>
-        </collision>    <visual>
-        <origin xyz="0 0 0" rpy="0 0 0"/>
-        <geometry>
-            <box size="0.04 0.01 0.01"/>
-        </geometry>
-        </visual>    <inertial>
-        <mass value="1e-5" />
-        <origin xyz="0 0 0" rpy="0 0 0"/>
-        <inertia ixx="1e-6" ixy="0" ixz="0" iyy="1e-6" iyz="0" izz="1e-6" />
-        </inertial>
-    </link>
+  <joint name="sonar_front_joint_left" type="fixed">
+    <axis xyz="0 1 0" />
+    <origin rpy="0 0 0.2" xyz="0.035 0.044 0.078" />
+    <parent link="base_link"/>
+    <child link="base_sonar_front_left"/>
+  </joint>
+  <link name="base_sonar_front_left">
+    <collision>
+      <origin xyz="0 0 0" rpy="0 0 0"/>
+      <geometry>
+          <box size="0.04 0.01 0.01"/>
+      </geometry>
+    </collision>
+    <visual>
+      <origin xyz="0 0 0" rpy="0 0 0"/>
+      <geometry>
+          <box size="0.04 0.01 0.01"/>
+      </geometry>
+    </visual>
+    <inertial>
+      <mass value="1e-5" />
+      <origin xyz="0 0 0" rpy="0 0 0"/>
+      <inertia ixx="1e-6" ixy="0" ixz="0" iyy="1e-6" iyz="0" izz="1e-6" />
+    </inertial>
+  </link>
+  <joint name="sonar_front_joint_right" type="fixed">
+    <axis xyz="0 1 0" />
+    <origin rpy="0 0 -0.2" xyz="0.035 -0.044 0.078" />
+    <parent link="base_link"/>
+    <child link="base_sonar_front_right"/>
+  </joint>
+  <link name="base_sonar_front_right">
+    <collision>
+      <origin xyz="0 0 0" rpy="0 0 0"/>
+      <geometry>
+        <box size="0.04 0.01 0.01"/>
+      </geometry>
+    </collision>
+    <visual>
+      <origin xyz="0 0 0" rpy="0 0 0"/>
+      <geometry>
+      <box size="0.04 0.01 0.01"/>
+      </geometry>
+    </visual>
+    <inertial>
+      <mass value="1e-5" />
+      <origin xyz="0 0 0" rpy="0 0 0"/>
+      <inertia ixx="1e-6" ixy="0" ixz="0" iyy="1e-6" iyz="0" izz="1e-6" />
+    </inertial>
+  </link>
 </robot>

Commit message: fake sonar

File: urdf/turtlebot3_burger_sonar.urdf.xacro (robot description, xacro)
@@ -194,3 +194,28 @@
     </inertial>
   </link>
+  <joint name="sonar_front_joint_middle" type="fixed">
+    <axis xyz="0 1 0" />
+    <origin rpy="0 0 0" xyz="0.035 0 0.078" />
+    <parent link="base_link"/>
+    <child link="base_sonar_front_middle"/>
+  </joint>
+  <link name="base_sonar_front_middle">
+    <collision>
+      <origin xyz="0 0 0" rpy="0 0 0"/>
+      <geometry>
+        <box size="0.04 0.01 0.01"/>
+      </geometry>
+    </collision>
+    <visual>
+      <origin xyz="0 0 0" rpy="0 0 0"/>
+      <geometry>
+      <box size="0.04 0.01 0.01"/>
+      </geometry>
+    </visual>
+    <inertial>
+      <mass value="1e-5" />
+      <origin xyz="0 0 0" rpy="0 0 0"/>
+      <inertia ixx="1e-6" ixy="0" ixz="0" iyy="1e-6" iyz="0" izz="1e-6" />
+    </inertial>
+  </link>
 </robot>

Commit message: Parametertuning

File: urdf/turtlebot3_burger_sonar.urdf.xacro (robot description, xacro)
@@ -146,5 +146,5 @@
   <joint name="sonar_front_joint_left" type="fixed">
     <axis xyz="0 1 0" />
-    <origin rpy="0 0 0.2" xyz="0.035 0.044 0.078" />
+    <origin rpy="0 0 0" xyz="0.035 0.044 0.078" />
     <parent link="base_link"/>
     <child link="base_sonar_front_left"/>
@@ -171,5 +171,5 @@
   <joint name="sonar_front_joint_right" type="fixed">
     <axis xyz="0 1 0" />
-    <origin rpy="0 0 -0.2" xyz="0.035 -0.044 0.078" />
+    <origin rpy="0 0 0" xyz="0.035 -0.044 0.078" />
     <parent link="base_link"/>
     <child link="base_sonar_front_right"/>
